Commit message: complete the robot and add the arm

File: course_1/src/my_robot_description/urdf/command_properties.xacro (robot description, xacro)
@@ -6,4 +6,10 @@
     <material name="grey">
         <color rgba="0.5 0.5 0.5 1" />
+    </material>
+    <material name="orange">
+        <color rgba="1.0 0.5 0 1" />
+    </material>
+    <material name="yellow">
+        <color rgba="1.0 1.0 0.5 1" />
     </material>
     <xacro:macro name="box_inertia" params="m l w h xyz rpy">

File: course_1/src/my_robot_description/urdf/my_robot.urdf.xacro (robot description, xacro)
@@ -5,3 +5,11 @@
     <xacro:include filename="mobile_base.xacro" />
     <xacro:include filename="mobile_base_gazebo.xacro" />
+    <xacro:include filename="arm.xacro" />
+    <xacro:include filename="arm_gazebo.xacro" />
+    <joint name="mobile_base_arm_joint" type="fixed">
+        <parent link="base_link" />
+        <child link="arm_base_link" />
+        <origin xyz="${base_length/4.0} 0 ${base_height}" rpy="0 0 0" />
+    </joint>
+    <!-- <xacro:include filename="camera.xacro" /> -->
 </robot>
